File: multilayer_pc.kicad_sch (KiCad schematic)
At the start: 60 parts, among them J1 USB_B_Micro, J10 Conn_01x04_Pin, J11 Conn_01x04_Pin, J12 Conn_01x04_Pin, J13 Conn_01x08, J14 Conn_01x08, J15 Conn_01x08, J16 Conn_01x08, J2 Jack-DC, J3 Screw_Terminal_01x02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

Commit message: Updated The PCB of the Project
Parts:
- removed R4, R5: 10k, symbol Device:R
- added J17: Conn_01x16, Connector_PinHeader_2.54mm:PinHeader_1x16_P2.54mm_Vertical, symbol Connector_Generic:Conn_01x16
- added J18: Conn_01x02, Connector_PinHeader_2.54mm:PinHeader_1x02_P2.54mm_Vertical, symbol Connector_Generic:Conn_01x02
- added R14, R15, R16, R17, R18, R19, R20: ~, Resistor_SMD:R_0805_2012Metric, symbol Device:R
- added RV1: R_Potentiometer, Potentiometer_THT:Potentiometer_Vishay_148-149_Single_Horizontal, symbol Device:R_Potentiometer
- added U5: HDSP-A153, Display_7Segment:HDSP-A151, symbol Display_Character:HDSP-A153
- C1, C10, C11, C12, C13, C14, C15, C16, C17, C18, C19, C2, C20, C21, C4, C5, C6, C7, C8, C9: footprint (none) -> Capacitor_SMD:C_0805_2012Metric
- J1: footprint (none) -> Connector_USB:USB_Micro-AB_Molex_47590-0001
- J10, J11, J12, J5, J8, J9: footprint (none) -> Connector:FanPinHeader_1x04_P2.54mm_Vertical
- J2: footprint (none) -> Connector_BarrelJack:BarrelJack_SwitchcraftConxall_RAPC10U_Horizontal
- J4: footprint (none) -> Connector_Molex:Molex_SL_171971-0002_1x02_P2.54mm_Vertical
- J6, J7: footprint (none) -> Connector:FanPinHeader_1x03_P2.54mm_Vertical
- R1, R10, R11, R12, R13, R2, R3, R6, R7, R8, R9: footprint (none) -> Resistor_SMD:R_0805_2012Metric
Connections:
- net +5V: now also J17.15 (Pin_15), J18.1 (Pin_1), RV1.1
- net GND: now also D1.2 (A), J17.1 (Pin_1), J17.16 (Pin_16), J17.5 (Pin_5), RV1.3, U5.1 (CC), U5.6 (CC); no longer D1.1 (K)
- net GPIO_1: now also D5.2 (A)
- net GPIO_10: now also J17.10 (Pin_10)
- net GPIO_11: now also J17.12 (Pin_12)
- net GPIO_14: now also J17.13 (Pin_13)
- net GPIO_15: now also J17.14 (Pin_14)
- net GPIO_25: now also R20.1
- net GPIO_26: now also J17.6 (Pin_6)
- net GPIO_3: now also D4.2 (A)
- net GPIO_32: now also R18.1
- net GPIO_33: now also R19.1
- net GPIO_34: now also R16.1
- net GPIO_35: now also R17.1
- net GPIO_36: now also R14.1
- net GPIO_39: now also R15.1
- net GPIO_4: now also J17.4 (Pin_4)
- net GPIO_6: now also J17.11 (Pin_11)
- net GPIO_7: now also J17.7 (Pin_7)
- net GPIO_8: now also J17.8 (Pin_8)
- net GPIO_9: now also J17.9 (Pin_9)
- net V_3.8V: no longer U3.4 (V3)
- net V_3.8V_OUT: now also U3.4 (V3)
- net at D3.1 (K), R3.2: now also D1.1 (K); no longer D1.2 (A)
- new net: R17.2, U5.5 (D)
- new net: R18.2, U5.4 (E)
- new net: J17.3 (Pin_3), RV1.2
- new net: R16.2, U5.8 (C)
- new net: R15.2, U5.9 (B)
- new net: R19.2, U5.2 (F)
- new net: J17.2 (Pin_2), J18.2 (Pin_2)
- new net: R20.2, U5.3 (G)
- new net: R14.2, U5.10 (A)
- no-connect marks 5 -> 6
Other:
- note added: "(Can also use Polarized capacitor if needed)"
- note added: "16x2 LCD Interface"
- note added: "7 Segment Display"
- note added: "CA (Common Anode) is avoided mostly CC (Common Cathode) is preffered"
- note added: "ESP32-WRoOM-32D Microcontroller"
- moved on the sheet: C4, C5, D1, U1, Y1
